Commit message: ros2_control_1

File: description/gazebo_control.xacro (robot description, xacro)
@@ -9,6 +9,6 @@
             <right_joint>right_back_wheel_joint</right_joint>
             <right_joint>right_front_wheel_joint</right_joint>
-            <wheel_separation>0.3194</wheel_separation>
-            <wheel_diameter>0.12</wheel_diameter>
+            <wheel_separation>0.3950</wheel_separation>
+            <wheel_diameter>0.14</wheel_diameter>
             <!--Limits-->
             <max_wheel_torque>200</max_wheel_torque>

File: description/robot.urdf.xacro (robot description, xacro)
@@ -3,4 +3,5 @@
     <xacro:include filename="robot_core.xacro" />
     <xacro:include filename="gazebo_control.xacro" />
+    <!--acro:include filename="ros2_control.xacro" /-->
     <xacro:include filename="lidar.xacro" />
     <xacro:include filename="camera.xacro" />

File: description/robot_core.xacro (robot description, xacro)
@@ -48,5 +48,5 @@
         <parent link="base_link"/>
         <child link="left_back_wheel"/>
-        <origin xyz="0.20495 0.1597 0" rpy="-${pi/2} 0 0"/>
+        <origin xyz="0.15495 0.1975 0" rpy="-${pi/2} 0 0"/>
         <axis xyz="0 0 1"/>
     </joint>
@@ -54,5 +54,5 @@
         <visual>
             <geometry>
-                <cylinder radius="0.06" length="0.04"/>
+                <cylinder radius="0.07" length="0.06"/>
             </geometry>
             <material name="blue"/>
@@ -60,8 +60,8 @@
         <collision>
             <geometry>
-                <cylinder radius="0.06" length="0.04"/>
+                <sphere radius="0.07"/>
             </geometry>
         </collision>
-        <xacro:inertial_cylinder mass="0.2" length="0.04" radius="0.06">
+        <xacro:inertial_cylinder mass="0.2" length="0.06" radius="0.07">
             <origin xyz="0 0 0" rpy="0 0 0"/>
         </xacro:inertial_cylinder>
@@ -74,5 +74,5 @@
         <parent link="base_link"/>
         <child link="right_back_wheel"/>
-        <origin xyz="0.20495 -0.1597 0" rpy="${pi/2} 0 0"/>
+        <origin xyz="0.15495 -0.1975 0" rpy="${pi/2} 0 0"/>
         <axis xyz="0 0 -1"/>
     </joint>
@@ -80,5 +80,5 @@
         <visual>
             <geometry>
-                <cylinder radius="0.06" length="0.04"/>
+                <cylinder radius="0.07" length="0.06"/>
             </geometry>
             <material name="blue"/>
@@ -86,8 +86,8 @@
         <collision>
             <geometry>
-                <cylinder radius="0.06" length="0.04"/>
+                <sphere radius="0.07"/>
             </geometry>
         </collision>
-        <xacro:inertial_cylinder mass="0.2" length="0.04" radius="0.06">
+        <xacro:inertial_cylinder mass="0.2" length="0.06" radius="0.07">
             <origin xyz="0 0 0" rpy="0 0 0"/>
         </xacro:inertial_cylinder>
@@ -100,5 +100,5 @@
         <parent link="base_link"/>
         <child link="left_front_wheel"/>
-        <origin xyz="-0.20495 0.1597 0" rpy="-${pi/2} 0 0"/>
+        <origin xyz="-0.15495 0.1975 0" rpy="-${pi/2} 0 0"/>
         <axis xyz="0 0 1"/>
     </joint>
@@ -106,5 +106,5 @@
         <visual>
             <geometry>
-                <cylinder radius="0.06" length="0.04"/>
+                <cylinder radius="0.07" length="0.06"/>
             </geometry>
             <material name="blue"/>
@@ -112,8 +112,8 @@
         <collision>
             <geometry>
-                <cylinder radius="0.06" length="0.04"/>
+                <sphere radius="0.07"/>
             </geometry>
         </collision>
-        <xacro:inertial_cylinder mass="0.2" length="0.04" radius="0.06">
+        <xacro:inertial_cylinder mass="0.2" length="0.06" radius="0.07">
             <origin xyz="0 0 0" rpy="0 0 0"/>
         </xacro:inertial_cylinder>
@@ -126,5 +126,5 @@
         <parent link="base_link"/>
         <child link="right_front_wheel"/>
-        <origin xyz="-0.20495 -0.1597 0" rpy="${pi/2} 0 0"/>
+        <origin xyz="-0.15495 -0.1975 0" rpy="${pi/2} 0 0"/>
         <axis xyz="0 0 -1"/>
     </joint>
@@ -132,5 +132,5 @@
         <visual>
             <geometry>
-                <cylinder radius="0.06" length="0.04"/>
+                <cylinder radius="0.07" length="0.06"/>
             </geometry>
             <material name="blue"/>
@@ -138,8 +138,8 @@
         <collision>
             <geometry>
-                <cylinder radius="0.06" length="0.04"/>
+                <sphere radius="0.07"/>
             </geometry>
         </collision>
-        <xacro:inertial_cylinder mass="0.2" length="0.04" radius="0.06">
+        <xacro:inertial_cylinder mass="0.2" length="0.06" radius="0.07">
             <origin xyz="0 0 0" rpy="0 0 0"/>
         </xacro:inertial_cylinder>
