Commit message: Gazebo tutorial done

File: description/robot_core.xacro (robot description, xacro)
@@ -41,4 +41,7 @@
         </xacro:inertial_box>
     </link>
+    <gazebo reference="chassis">
+        <material>Gazebo/White</material>
+    </gazebo>
     <!-- Left Back wheel link-->
     <joint name="left_back_wheel_joint" type="continuous">
@@ -64,4 +67,7 @@
         </xacro:inertial_cylinder>
     </link>
+    <gazebo reference="left_back_wheel">
+        <material>Gazebo/Blue</material>
+    </gazebo>
     <!-- Right Back wheel link-->
     <joint name="right_back_wheel_joint" type="continuous">
@@ -87,4 +93,7 @@
         </xacro:inertial_cylinder>
     </link>
+    <gazebo reference="right_back_wheel">
+        <material>Gazebo/Blue</material>
+    </gazebo>
     <!-- Left front wheel link-->
     <joint name="left_front_wheel_joint" type="continuous">
@@ -110,4 +119,7 @@
         </xacro:inertial_cylinder>
     </link>
+    <gazebo reference="left_front_wheel">
+        <material>Gazebo/Blue</material>
+    </gazebo>
     <!-- Right front wheel link-->
     <joint name="right_front_wheel_joint" type="continuous">
@@ -133,3 +145,6 @@
         </xacro:inertial_cylinder>
     </link>
+    <gazebo reference="right_front_wheel">
+        <material>Gazebo/Blue</material>
+    </gazebo>
 </robot>

Commit message: lol3

File: description/robot_core.xacro (robot description, xacro)
@@ -70,4 +70,30 @@
         <material>Gazebo/Blue</material>
     </gazebo>
+    <!-- Left front wheel link-->
+    <joint name="left_front_wheel_joint" type="continuous">
+        <parent link="base_link"/>
+        <child link="left_front_wheel"/>
+        <origin xyz="-0.13 0.1975 0" rpy="-${pi/2} 0 0"/>
+        <axis xyz="0 0 1"/>
+    </joint>
+    <link name="left_front_wheel">
+        <visual>
+            <geometry>
+                <cylinder radius="0.07" length="0.06"/>
+            </geometry>
+            <material name="blue"/>
+        </visual>
+        <collision>
+            <geometry>
+                <sphere radius="0.07"/>
+            </geometry>
+        </collision>
+        <xacro:inertial_cylinder mass="0.2" length="0.06" radius="0.07">
+            <origin xyz="0 0 0" rpy="0 0 0"/>
+        </xacro:inertial_cylinder>
+    </link>
+    <gazebo reference="left_front_wheel">
+        <material>Gazebo/Blue</material>
+    </gazebo>
     <!-- Right Back wheel link-->
     <joint name="right_back_wheel_joint" type="continuous">
@@ -94,30 +120,4 @@
     </link>
     <gazebo reference="right_back_wheel">
-        <material>Gazebo/Blue</material>
-    </gazebo>
-    <!-- Left front wheel link-->
-    <joint name="left_front_wheel_joint" type="continuous">
-        <parent link="base_link"/>
-        <child link="left_front_wheel"/>
-        <origin xyz="-0.13 0.1975 0" rpy="-${pi/2} 0 0"/>
-        <axis xyz="0 0 1"/>
-    </joint>
-    <link name="left_front_wheel">
-        <visual>
-            <geometry>
-                <cylinder radius="0.07" length="0.06"/>
-            </geometry>
-            <material name="blue"/>
-        </visual>
-        <collision>
-            <geometry>
-                <sphere radius="0.07"/>
-            </geometry>
-        </collision>
-        <xacro:inertial_cylinder mass="0.2" length="0.06" radius="0.07">
-            <origin xyz="0 0 0" rpy="0 0 0"/>
-        </xacro:inertial_cylinder>
-    </link>
-    <gazebo reference="left_front_wheel">
         <material>Gazebo/Blue</material>
     </gazebo>

File: description/ros2_control.xacro (robot description, xacro)
@@ -1,78 +1,91 @@
 <?xml version="1.0"?>
 <robot xmlns:xacro="http://www.ros.org/wiki/xacro" >
-    <ros2_control name="GazeboSystem" type="system">
-        <hardware>
-            <plugin>gazebo_ros2_control/GazeboSystem</plugin>
-        </hardware>
-        <joint name="left_back_wheel_joint">
-            <command_interface name ="velocity">
-                <param name="min">-50</param>
-                <param name="max">50</param>
-            </command_interface>
-            <state_interface name="velocity"/>
-            <state_interface name="position"/>
-        </joint>
-        <joint name="right_back_wheel_joint">
-            <command_interface name ="velocity">
-                <param name="min">-50</param>
-                <param name="max">50</param>
-            </command_interface>
-            <state_interface name="velocity"/>
-            <state_interface name="position"/>
-        </joint>
-        <joint name="left_front_wheel_joint">
-            <command_interface name ="velocity">
-                <param name="min">-50</param>
-                <param name="max">50</param>
-            </command_interface>
-            <state_interface name="velocity"/>
-            <state_interface name="position"/>
-        </joint>
-        <joint name="right_front_wheel_joint">
-            <command_interface name ="velocity">
-                <param name="min">-50</param>
-                <param name="max">50</param>
-            </command_interface>
-            <state_interface name="velocity"/>
-            <state_interface name="position"/>
-        </joint>
-    </ros2_control>
+    <xacro:unless value="$(arg sim_mode)">
+        <ros2_control name="RealRobot" type="system">
+            <hardware>
+                <plugin>diffdrive_arduino/DiffDriveArduino</plugin>
+                <param name="left_back_wheel_name">left_back_wheel_joint</param>
+                <param name="left_front_wheel_name">left_front_wheel_joint</param>
+                <param name="right_back_wheel_name">right_back_wheel_joint</param>
+                <param name="right_front_wheel_name">right_front_wheel_joint</param>
+                <param name="loop_rate">30</param>
+                <param name="device">/dev/ttyACM0</param>
+                <param name="baud_rate">57600</param>
+                <param name="timeout">1000</param>
+                <param name="enc_counts_per_rev">3436</param>
+            </hardware>
+            <joint name="left_back_wheel_joint">
+                <command_interface name ="velocity">
+                    <param name="min">-50</param>
+                    <param name="max">50</param>
+                </command_interface>
+                <state_interface name="velocity"/>
+                <state_interface name="position"/>
+            </joint>
+            <joint name="left_front_wheel_joint">
+                <command_interface name ="velocity">
+                    <param name="min">-50</param>
+                    <param name="max">50</param>
+                </command_interface>
+                <state_interface name="velocity"/>
+                <state_interface name="position"/>
+            </joint>
+            <joint name="right_back_wheel_joint">
+                <command_interface name ="velocity">
+                    <param name="min">-50</param>
+                    <param name="max">50</param>
+                </command_interface>
+                <state_interface name="velocity"/>
+                <state_interface name="position"/>
+            </joint>
+            <joint name="right_front_wheel_joint">
+                <command_interface name ="velocity">
+                    <param name="min">-50</param>
+                    <param name="max">50</param>
+                </command_interface>
+                <state_interface name="velocity"/>
+                <state_interface name="position"/>
+            </joint>
+        </ros2_control>
+    </xacro:unless>
+    <xacro:if value="$(arg sim_mode)">
         <ros2_control name="GazeboSystem" type="system">
-        <hardware>
-            <plugin>gazebo_ros2_control/GazeboSystem</plugin>
-        </hardware>
-        <joint name="left_back_wheel_joint">
-            <command_interface name ="velocity">
-                <param name="min">-50</param>
-                <param name="max">50</param>
-            </command_interface>
-            <state_interface name="velocity"/>
-            <state_interface name="position"/>
-        </joint>
-        <joint name="right_back_wheel_joint">
-            <command_interface name ="velocity">
-                <param name="min">-50</param>
-                <param name="max">50</param>
-            </command_interface>
-            <state_interface name="velocity"/>
-            <state_interface name="position"/>
-        </joint>
-        <joint name="left_front_wheel_joint">
-            <command_interface name ="velocity">
-                <param name="min">-50</param>
-                <param name="max">50</param>
-            </command_interface>
-            <state_interface name="velocity"/>
-            <state_interface name="position"/>
-        </joint>
-        <joint name="right_front_wheel_joint">
-            <command_interface name ="velocity">
-                <param name="min">-50</param>
-                <param name="max">50</param>
-            </command_interface>
-            <state_interface name="velocity"/>
-            <state_interface name="position"/>
-        </joint>
-    </ros2_control>
+            <hardware>
+                <plugin>gazebo_ros2_control/GazeboSystem</plugin>
+            </hardware>
+            <joint name="left_back_wheel_joint">
+                <command_interface name ="velocity">
+                    <param name="min">-50</param>
+                    <param name="max">50</param>
+                </command_interface>
+                <state_interface name="velocity"/>
+                <state_interface name="position"/>
+            </joint>
+            <joint name="right_back_wheel_joint">
+                <command_interface name ="velocity">
+                    <param name="min">-50</param>
+                    <param name="max">50</param>
+                </command_interface>
+                <state_interface name="velocity"/>
+                <state_interface name="position"/>
+            </joint>
+            <joint name="left_front_wheel_joint">
+                <command_interface name ="velocity">
+                    <param name="min">-50</param>
+                    <param name="max">50</param>
+                </command_interface>
+                <state_interface name="velocity"/>
+                <state_interface name="position"/>
+            </joint>
+            <joint name="right_front_wheel_joint">
+                <command_interface name ="velocity">
+                    <param name="min">-50</param>
+                    <param name="max">50</param>
+                </command_interface>
+                <state_interface name="velocity"/>
+                <state_interface name="position"/>
+            </joint>
+        </ros2_control>
+    </xacro:if>
     <gazebo>
         <plugin name="gazebo_ros2_control" filename="libgazebo_ros2_control.so">

Commit message: fixing URDF to new design along with simulation fixes

File: description/robot_core.xacro (robot description, xacro)
@@ -48,20 +48,20 @@
         <parent link="base_link"/>
         <child link="left_back_wheel"/>
-        <origin xyz="0.13 0.1975 0" rpy="-${pi/2} 0 0"/>
+        <origin xyz="0 0.16 0" rpy="-${pi/2} 0 0"/>
         <axis xyz="0 0 1"/>
     </joint>
     <link name="left_back_wheel">
-        <visual>
-            <geometry>
-                <cylinder radius="0.07" length="0.06"/>
-            </geometry>
-            <material name="blue"/>
-        </visual>
-        <collision>
-            <geometry>
-                <sphere radius="0.07"/>
-            </geometry>
-        </collision>
-        <xacro:inertial_cylinder mass="0.2" length="0.06" radius="0.07">
+        <!--visual>
+            <geometry>
+                <cylinder radius="0.035" length="0.02"/>
+            </geometry>
+            <material name="blue"/>
+        </visual-->
+        <!--collision>
+            <geometry>
+                <sphere radius="0.035"/>
+            </geometry>
+        </collision-->
+        <xacro:inertial_cylinder mass="0.2" length="0.02" radius="0.035">
             <origin xyz="0 0 0" rpy="0 0 0"/>
         </xacro:inertial_cylinder>
@@ -74,5 +74,5 @@
         <parent link="base_link"/>
         <child link="left_front_wheel"/>
-        <origin xyz="-0.13 0.1975 0" rpy="-${pi/2} 0 0"/>
+        <origin xyz="0.13 0.16 0" rpy="-${pi/2} 0 0"/>
         <axis xyz="0 0 1"/>
     </joint>
@@ -80,14 +80,14 @@
         <visual>
             <geometry>
-                <cylinder radius="0.07" length="0.06"/>
-            </geometry>
-            <material name="blue"/>
-        </visual>
-        <collision>
-            <geometry>
-                <sphere radius="0.07"/>
-            </geometry>
-        </collision>
-        <xacro:inertial_cylinder mass="0.2" length="0.06" radius="0.07">
+                <cylinder radius="0.035" length="0.02"/>
+            </geometry>
+            <material name="blue"/>
+        </visual>
+        <collision>
+            <geometry>
+                <sphere radius="0.035"/>
+            </geometry>
+        </collision>
+        <xacro:inertial_cylinder mass="0.2" length="0.02" radius="0.035">
             <origin xyz="0 0 0" rpy="0 0 0"/>
         </xacro:inertial_cylinder>
@@ -100,20 +100,20 @@
         <parent link="base_link"/>
         <child link="right_back_wheel"/>
-        <origin xyz="0.13 -0.1975 0" rpy="${pi/2} 0 0"/>
+        <origin xyz="0 -0.16 0" rpy="${pi/2} 0 0"/>
         <axis xyz="0 0 -1"/>
     </joint>
     <link name="right_back_wheel">
-        <visual>
-            <geometry>
-                <cylinder radius="0.07" length="0.06"/>
-            </geometry>
-            <material name="blue"/>
-        </visual>
-        <collision>
-            <geometry>
-                <sphere radius="0.07"/>
-            </geometry>
-        </collision>
-        <xacro:inertial_cylinder mass="0.2" length="0.06" radius="0.07">
+        <!--visual>
+            <geometry>
+                <cylinder radius="0.035" length="0.02"/>
+            </geometry>
+            <material name="blue"/>
+        </visual-->
+        <!--collision>
+            <geometry>
+                <sphere radius="0.035"/>
+            </geometry>
+        </collision-->
+        <xacro:inertial_cylinder mass="0.2" length="0.02" radius="0.035">
             <origin xyz="0 0 0" rpy="0 0 0"/>
         </xacro:inertial_cylinder>
@@ -126,5 +126,5 @@
         <parent link="base_link"/>
         <child link="right_front_wheel"/>
-        <origin xyz="-0.13 -0.1975 0" rpy="${pi/2} 0 0"/>
+        <origin xyz="0.13 -0.16 0" rpy="${pi/2} 0 0"/>
         <axis xyz="0 0 -1"/>
     </joint>
@@ -132,14 +132,14 @@
         <visual>
             <geometry>
-                <cylinder radius="0.07" length="0.06"/>
-            </geometry>
-            <material name="blue"/>
-        </visual>
-        <collision>
-            <geometry>
-                <sphere radius="0.07"/>
-            </geometry>
-        </collision>
-        <xacro:inertial_cylinder mass="0.2" length="0.06" radius="0.07">
+                <cylinder radius="0.035" length="0.02"/>
+            </geometry>
+            <material name="blue"/>
+        </visual>
+        <collision>
+            <geometry>
+                <sphere radius="0.035"/>
+            </geometry>
+        </collision>
+        <xacro:inertial_cylinder mass="0.2" length="0.02" radius="0.035">
             <origin xyz="0 0 0" rpy="0 0 0"/>
         </xacro:inertial_cylinder>
@@ -148,3 +148,57 @@
         <material>Gazebo/Blue</material>
     </gazebo>
+    <!--Left Caster wheel Link-->
+    <joint name="left_caster_wheel_joint" type="fixed">
+        <parent link="chassis"/>
+        <child link="left_caster_wheel"/>
+        <origin xyz="0.13 0.09 0"/>
+    </joint>
+    <link name="left_caster_wheel">
+        <visual>
+            <geometry>
+                <sphere radius="0.035"/>
+            </geometry>
+            <material name="black"/>
+        </visual>
+        <collision>
+            <geometry>
+                <sphere radius="0.035"/>
+            </geometry>
+        </collision>
+        <xacro:inertial_sphere mass="0.2" radius="0.035">
+            <origin xyz="0 0 0" rpy="0 0 0"/>
+        </xacro:inertial_sphere>
+    </link>
+    <gazebo reference="left_caster_wheel">
+        <material>Gazebo/Black</material>
+        <mu1 value="0.001"/>
+        <mu2 value="0.001"/>
+    </gazebo>
+    <!--Right Caster wheel Link-->
+    <joint name="right_caster_wheel_joint" type="fixed">
+        <parent link="chassis"/>
+        <child link="right_caster_wheel"/>
+        <origin xyz="0.13 -0.09 0"/>
+    </joint>
+    <link name="right_caster_wheel">
+        <visual>
+            <geometry>
+                <sphere radius="0.035"/>
+            </geometry>
+            <material name="black"/>
+        </visual>
+        <collision>
+            <geometry>
+                <sphere radius="0.035"/>
+            </geometry>
+        </collision>
+        <xacro:inertial_sphere mass="0.2" radius="0.035">
+            <origin xyz="0 0 0" rpy="0 0 0"/>
+        </xacro:inertial_sphere>
+    </link>
+    <gazebo reference="right_caster_wheel">
+        <material>Gazebo/Black</material>
+        <mu1 value="0.001"/>
+        <mu2 value="0.001"/>
+    </gazebo>
 </robot>

Commit message: SLAM

File: description/robot_core.xacro (robot description, xacro)
@@ -17,4 +17,11 @@
     <link name="base_link">
     </link>
+    <joint name="base_footprint_joint" type="fixed">
+        <parent link="base_link"/>
+        <child link="base_footprint"/>
+        <origin xyz="0 0 0" rpy="0 0 0"/>
+    </joint>
+    <link name="base_footprint">
+    </link>
     <!-- Chassis Link -->
     <joint name="chassis_joint" type="fixed">
