Commit message: changes as of march 25, 2024

File: description/camera.xacro (robot description, xacro)
@@ -4,5 +4,5 @@
         <parent link="chassis"/>
         <child link="camera_link"/>
-        <origin xyz="0.4749 0 0.3931" rpy="0 0 0"/>
+        <origin xyz="0.4 0 0.625" rpy="0 0 0"/>
     </joint>
     <link name="camera_link">

File: description/lidar.xacro (robot description, xacro)
@@ -4,5 +4,5 @@
         <parent link="chassis"/>
         <child link="laser_frame"/>
-        <origin xyz="0.23495 0 0.6931" rpy="0 0 0"/>
+        <origin xyz="0.23 0 0.65" rpy="0 0 0"/>
     </joint>
     <link name="laser_frame">

File: description/robot.urdf.xacro (robot description, xacro)
@@ -1,7 +1,12 @@
 <?xml version="1.0"?>
 <robot xmlns:xacro="http://www.ros.org/wiki/xacro"  name="robot">
+    <xacro:arg name="use_ros2_control" default="true"/>
     <xacro:include filename="robot_core.xacro" />
-    <xacro:include filename="gazebo_control.xacro" />
-    <!--acro:include filename="ros2_control.xacro" /-->
+    <xacro:if value="$(arg use_ros2_control)">
+        <xacro:include filename="ros2_control.xacro" />
+    </xacro:if>
+    <xacro:unless value="$(arg use_ros2_control)">
+        <xacro:include filename="gazebo_control.xacro" />
+    </xacro:unless>
     <xacro:include filename="lidar.xacro" />
     <xacro:include filename="camera.xacro" />

File: description/robot_core.xacro (robot description, xacro)
@@ -21,22 +21,22 @@
         <parent link="base_link"/>
         <child link="chassis"/>
-        <origin xyz="-0.23495 0 0"/>
+        <origin xyz="-0.23 0 0"/>
     </joint>
     <link name="chassis">
         <visual>
-            <origin xyz="0.23495 0 0.33655"/>
+            <origin xyz="0.23 0 0.305"/>
             <geometry>
-                <box size="0.4699 0.2794  0.6731"/>
+                <box size="0.46 0.285  0.61"/>
             </geometry>
             <material name="white"/>
         </visual>
         <collision>
-            <origin xyz="0.23495 0 0.33655"/>
+            <origin xyz="0.23 0 0.305"/>
             <geometry>
-                <box size="0.4699 0.2794  0.6731"/>
+                <box size="0.46 0.285  0.61"/>
             </geometry>
         </collision>
-        <xacro:inertial_box mass="3.175" x="0.4699" y="0.2794" z="0.6731">
-            <origin xyz="0.23495 0 0.33655" rpy="0 0 0"/>
+        <xacro:inertial_box mass="3.175" x="0.46" y="0.285" z="0.61">
+            <origin xyz="0.23 0 0.305" rpy="0 0 0"/>
         </xacro:inertial_box>
     </link>
@@ -48,5 +48,5 @@
         <parent link="base_link"/>
         <child link="left_back_wheel"/>
-        <origin xyz="0.15495 0.1975 0" rpy="-${pi/2} 0 0"/>
+        <origin xyz="0.13 0.1975 0" rpy="-${pi/2} 0 0"/>
         <axis xyz="0 0 1"/>
     </joint>
@@ -74,5 +74,5 @@
         <parent link="base_link"/>
         <child link="right_back_wheel"/>
-        <origin xyz="0.15495 -0.1975 0" rpy="${pi/2} 0 0"/>
+        <origin xyz="0.13 -0.1975 0" rpy="${pi/2} 0 0"/>
         <axis xyz="0 0 -1"/>
     </joint>
@@ -100,5 +100,5 @@
         <parent link="base_link"/>
         <child link="left_front_wheel"/>
-        <origin xyz="-0.15495 0.1975 0" rpy="-${pi/2} 0 0"/>
+        <origin xyz="-0.13 0.1975 0" rpy="-${pi/2} 0 0"/>
         <axis xyz="0 0 1"/>
     </joint>
@@ -126,5 +126,5 @@
         <parent link="base_link"/>
         <child link="right_front_wheel"/>
-        <origin xyz="-0.15495 -0.1975 0" rpy="${pi/2} 0 0"/>
+        <origin xyz="-0.13 -0.1975 0" rpy="${pi/2} 0 0"/>
         <axis xyz="0 0 -1"/>
     </joint>

Commit message: final commit for VY05

File: description/camera.xacro (robot description, xacro)
@@ -4,5 +4,5 @@
         <parent link="chassis"/>
         <child link="camera_link"/>
-        <origin xyz="0.4 0 0.625" rpy="0 0 0"/>
+        <origin xyz="0.4 0 0.375" rpy="0 0 0"/>
     </joint>
     <link name="camera_link">

File: description/lidar.xacro (robot description, xacro)
@@ -4,5 +4,5 @@
         <parent link="chassis"/>
         <child link="laser_frame"/>
-        <origin xyz="0.23 0 0.65" rpy="0 0 0"/>
+        <origin xyz="0.23 0 0.40" rpy="0 0 0"/>
     </joint>
     <link name="laser_frame">

File: description/robot.urdf.xacro (robot description, xacro)
@@ -2,5 +2,5 @@
 <robot xmlns:xacro="http://www.ros.org/wiki/xacro"  name="robot">
     <xacro:arg name="use_ros2_control" default="true"/>
-    <xacro:arg name="sim_mode" default="true"/>
+    <xacro:arg name="sim_mode" default="false"/>
     <xacro:include filename="robot_core.xacro" />
     <xacro:if value="$(arg use_ros2_control)">
@@ -12,4 +12,3 @@
     <xacro:include filename="lidar.xacro" />
     <xacro:include filename="camera.xacro" />
-    <!-- <xacro:include filename="depth_camera.xacro" /> -->
 </robot>

File: description/robot_core.xacro (robot description, xacro)
@@ -32,17 +32,17 @@
     <link name="chassis">
         <visual>
-            <origin xyz="0.23 0 0.305"/>
-            <geometry>
-                <box size="0.46 0.285  0.61"/>
+            <origin xyz="0.23 0 0.18"/>
+            <geometry>
+                <box size="0.46 0.285  0.36"/>
             </geometry>
             <material name="white"/>
         </visual>
         <collision>
-            <origin xyz="0.23 0 0.305"/>
-            <geometry>
-                <box size="0.46 0.285  0.61"/>
-            </geometry>
-        </collision>
-        <xacro:inertial_box mass="3.175" x="0.46" y="0.285" z="0.61">
+            <origin xyz="0.23 0 0.18"/>
+            <geometry>
+                <box size="0.46 0.285  0.36"/>
+            </geometry>
+        </collision>
+        <xacro:inertial_box mass="8" x="0.46" y="0.285" z="0.36">
             <origin xyz="0.23 0 0.305" rpy="0 0 0"/>
         </xacro:inertial_box>

File: description/ros2_control.xacro (robot description, xacro)
@@ -4,5 +4,5 @@
         <ros2_control name="RealRobot" type="system">
             <hardware>
-                <plugin>diffdrive_arduino/DiffDriveArduino</plugin>
+                <plugin>diffdrive_arduino/DiffDriveArduinoHardware</plugin>
                 <param name="left_back_wheel_name">left_back_wheel_joint</param>
                 <param name="left_front_wheel_name">left_front_wheel_joint</param>
@@ -12,6 +12,6 @@
                 <param name="device">/dev/ttyACM0</param>
                 <param name="baud_rate">57600</param>
-                <param name="timeout">1000</param>
-                <param name="enc_counts_per_rev">3436</param>
+                <param name="timeout_ms">1000</param>
+                <param name="enc_counts_per_rev">2500</param>
             </hardware>
             <joint name="left_back_wheel_joint">
@@ -20,6 +20,6 @@
                     <param name="max">50</param>
                 </command_interface>
+                <state_interface name="position"/>
                 <state_interface name="velocity"/>
-                <state_interface name="position"/>
             </joint>
             <joint name="left_front_wheel_joint">
@@ -28,6 +28,6 @@
                     <param name="max">50</param>
                 </command_interface>
+                <state_interface name="position"/>
                 <state_interface name="velocity"/>
-                <state_interface name="position"/>
             </joint>
             <joint name="right_back_wheel_joint">
@@ -36,6 +36,6 @@
                     <param name="max">50</param>
                 </command_interface>
+                <state_interface name="position"/>
                 <state_interface name="velocity"/>
-                <state_interface name="position"/>
             </joint>
             <joint name="right_front_wheel_joint">
@@ -44,6 +44,6 @@
                     <param name="max">50</param>
                 </command_interface>
+                <state_interface name="position"/>
                 <state_interface name="velocity"/>
-                <state_interface name="position"/>
             </joint>
         </ros2_control>
@@ -59,6 +59,6 @@
                     <param name="max">50</param>
                 </command_interface>
+                <state_interface name="position"/>
                 <state_interface name="velocity"/>
-                <state_interface name="position"/>
             </joint>
             <joint name="right_back_wheel_joint">
@@ -67,6 +67,6 @@
                     <param name="max">50</param>
                 </command_interface>
+                <state_interface name="position"/>
                 <state_interface name="velocity"/>
-                <state_interface name="position"/>
             </joint>
             <joint name="left_front_wheel_joint">
@@ -75,6 +75,6 @@
                     <param name="max">50</param>
                 </command_interface>
+                <state_interface name="position"/>
                 <state_interface name="velocity"/>
-                <state_interface name="position"/>
             </joint>
             <joint name="right_front_wheel_joint">
@@ -83,6 +83,6 @@
                     <param name="max">50</param>
                 </command_interface>
+                <state_interface name="position"/>
                 <state_interface name="velocity"/>
-                <state_interface name="position"/>
             </joint>
         </ros2_control>
